Commit message: Add files via upload

File: backups/lunarbot/urdf/lunarbot.urdf.xacro (robot description, xacro)
@@ -13,7 +13,4 @@
     <color rgba="1 1 1 1"/>
   </material>
-  <!--Add <gazebo> element to <robot>, <link>, and <joint> elements-->
-  <gazebo>
-	</gazebo>
   <!--Links-->
   <!--Body(base_link)-->
@@ -38,6 +35,4 @@
       <inertia ixx="4.05" ixy="0" ixz="0" iyy="9.82" iyz="0" izz="12.25"/>
     </inertial>
-    <gazebo>
-		</gazebo>
   </link>
   <link name="link_0">
@@ -59,6 +54,4 @@
       <inertia ixx=".14" ixy="0" ixz="0" iyy="0.24" iyz="0" izz=".14"/>
     </inertial>
-    <gazebo>
-			</gazebo>
   </link>
   <joint name="joint_0" type="continuous">
@@ -67,6 +60,4 @@
     <axis xyz="0 1 0"/>
     <origin rpy="0 0 0" xyz="0.3 0.375 -0.075"/>
-    <gazebo>
-			</gazebo>
   </joint>
   <link name="link_1">
@@ -88,6 +79,4 @@
       <inertia ixx=".14" ixy="0" ixz="0" iyy="0.24" iyz="0" izz=".14"/>
     </inertial>
-    <gazebo>
-			</gazebo>
   </link>
   <joint name="joint_1" type="continuous">
@@ -96,6 +85,4 @@
     <axis xyz="0 1 0"/>
     <origin rpy="0 0 0" xyz="0.3 -0.375 -0.075"/>
-    <gazebo>
-			</gazebo>
   </joint>
   <link name="link_2">
@@ -117,6 +104,4 @@
       <inertia ixx=".14" ixy="0" ixz="0" iyy="0.24" iyz="0" izz=".14"/>
     </inertial>
-    <gazebo>
-			</gazebo>
   </link>
   <joint name="joint_2" type="continuous">
@@ -125,6 +110,4 @@
     <axis xyz="0 1 0"/>
     <origin rpy="0 0 0" xyz="-0.3 0.375 -0.075"/>
-    <gazebo>
-			</gazebo>
   </joint>
   <link name="link_3">
@@ -146,6 +129,4 @@
       <inertia ixx=".14" ixy="0" ixz="0" iyy="0.24" iyz="0" izz=".14"/>
     </inertial>
-    <gazebo>
-			</gazebo>
   </link>
   <joint name="joint_3" type="continuous">
@@ -154,6 +135,10 @@
     <axis xyz="0 1 0"/>
     <origin rpy="0 0 0" xyz="-0.3 -0.375 -0.075"/>
-    <gazebo>
-			</gazebo>
   </joint>
+  <!--Plugin ties Gazebo to ROS-->
+  <gazebo>
+    <plugin filename="libgazebo_ros_control.so" name="gazebo_ros_control">
+      <robotNamespace>/</robotNamespace>
+    </plugin>
+  </gazebo>
 </robot>

File: backups/lunarbot/urdf/lunarbot.xacro (robot description, xacro)
@@ -9,7 +9,4 @@
     <color rgba="1 1 1 1"/>
   </material>
-	<!--Add <gazebo> element to <robot>, <link>, and <joint> elements-->
-	<gazebo>
-	</gazebo>
   <!--Xacro Macros-->
   <!--Body Macros-->
@@ -38,6 +35,4 @@
         <inertia ixx=".14" ixy="0" ixz="0" iyy="0.24" iyz="0" izz=".14"/>
       </inertial>
-			<gazebo>
-			</gazebo>
     </link>
     <joint name="joint_${suffix}" type="continuous">
@@ -46,6 +41,4 @@
       <axis xyz="0 1 0"/>
       <origin rpy="0 0 0" xyz="${reflect_x * 0.3} ${reflect_y * 0.375} ${reflect_z * 0.075}"/>
-			<gazebo>
-			</gazebo>
     </joint>
   </xacro:macro>
@@ -72,6 +65,4 @@
       <inertia ixx="4.05" ixy="0" ixz="0" iyy="9.82" iyz="0" izz="12.25"/>
     </inertial>
-		<gazebo>
-		</gazebo>
   </link>
   <!--wheel/joint_0-->
@@ -83,3 +74,9 @@
   <!--wheel/joint_3-->
   <xacro:wheel suffix="3" reflect_x="-1" reflect_y="-1" reflect_z="-1" />
+	<!--Plugin ties Gazebo to ROS-->
+	<gazebo>
+		<plugin name="gazebo_ros_control" filename="libgazebo_ros_control.so">
+			<robotNamespace>/</robotNamespace>
+		</plugin>
+	</gazebo>
 </robot>

Commit message: Add files via upload

File: backups/lunarbot/urdf/lunarbot.urdf.xacro (robot description, xacro)
@@ -35,4 +35,7 @@
       <inertia ixx="4.05" ixy="0" ixz="0" iyy="9.82" iyz="0" izz="12.25"/>
     </inertial>
+    <gazebo>
+      <material>Gazebo/Grey</material>
+    </gazebo>
   </link>
   <link name="link_0">
@@ -61,4 +64,22 @@
     <origin rpy="0 0 0" xyz="0.3 0.375 -0.075"/>
   </joint>
+  <!--Connects Gazebo to ROS Controls-->
+  <transmission name="joint_0_wheel_trans">
+    <type>transmission_interface/SimpleTransmission</type>
+    <actuator name="joint_0_wheel_motor">
+      <mechanicalReduction>1</mechanicalReduction>
+    </actuator>
+    <joint name="joint_0">
+      <hardwareInterface>hardware_interface/VelocityJointInterface</hardwareInterface>
+    </joint>
+  </transmission>
+  <!--Some extra Gazebo details-->
+  <gazebo reference="link_0">
+    <mu1 value="200.0"/>
+    <mu2 value="100.0"/>
+    <kp value="10000000.0"/>
+    <kd value="1.0"/>
+    <material>Gazebo/Blue</material>
+  </gazebo>
   <link name="link_1">
     <visual>
@@ -86,4 +107,22 @@
     <origin rpy="0 0 0" xyz="0.3 -0.375 -0.075"/>
   </joint>
+  <!--Connects Gazebo to ROS Controls-->
+  <transmission name="joint_1_wheel_trans">
+    <type>transmission_interface/SimpleTransmission</type>
+    <actuator name="joint_1_wheel_motor">
+      <mechanicalReduction>1</mechanicalReduction>
+    </actuator>
+    <joint name="joint_1">
+      <hardwareInterface>hardware_interface/VelocityJointInterface</hardwareInterface>
+    </joint>
+  </transmission>
+  <!--Some extra Gazebo details-->
+  <gazebo reference="link_1">
+    <mu1 value="200.0"/>
+    <mu2 value="100.0"/>
+    <kp value="10000000.0"/>
+    <kd value="1.0"/>
+    <material>Gazebo/Blue</material>
+  </gazebo>
   <link name="link_2">
     <visual>
@@ -111,4 +150,22 @@
     <origin rpy="0 0 0" xyz="-0.3 0.375 -0.075"/>
   </joint>
+  <!--Connects Gazebo to ROS Controls-->
+  <transmission name="joint_2_wheel_trans">
+    <type>transmission_interface/SimpleTransmission</type>
+    <actuator name="joint_2_wheel_motor">
+      <mechanicalReduction>1</mechanicalReduction>
+    </actuator>
+    <joint name="joint_2">
+      <hardwareInterface>hardware_interface/VelocityJointInterface</hardwareInterface>
+    </joint>
+  </transmission>
+  <!--Some extra Gazebo details-->
+  <gazebo reference="link_2">
+    <mu1 value="200.0"/>
+    <mu2 value="100.0"/>
+    <kp value="10000000.0"/>
+    <kd value="1.0"/>
+    <material>Gazebo/Blue</material>
+  </gazebo>
   <link name="link_3">
     <visual>
@@ -136,5 +193,23 @@
     <origin rpy="0 0 0" xyz="-0.3 -0.375 -0.075"/>
   </joint>
-  <!--Plugin ties Gazebo to ROS-->
+  <!--Connects Gazebo to ROS Controls-->
+  <transmission name="joint_3_wheel_trans">
+    <type>transmission_interface/SimpleTransmission</type>
+    <actuator name="joint_3_wheel_motor">
+      <mechanicalReduction>1</mechanicalReduction>
+    </actuator>
+    <joint name="joint_3">
+      <hardwareInterface>hardware_interface/VelocityJointInterface</hardwareInterface>
+    </joint>
+  </transmission>
+  <!--Some extra Gazebo details-->
+  <gazebo reference="link_3">
+    <mu1 value="200.0"/>
+    <mu2 value="100.0"/>
+    <kp value="10000000.0"/>
+    <kd value="1.0"/>
+    <material>Gazebo/Blue</material>
+  </gazebo>
+  <!--Gazebo plugin for ROS controls-->
   <gazebo>
     <plugin filename="libgazebo_ros_control.so" name="gazebo_ros_control">

File: backups/lunarbot/urdf/lunarbot.xacro (robot description, xacro)
@@ -42,4 +42,22 @@
       <origin rpy="0 0 0" xyz="${reflect_x * 0.3} ${reflect_y * 0.375} ${reflect_z * 0.075}"/>
     </joint>
+    <!--Connects Gazebo to ROS Controls-->
+    <transmission name="joint_${suffix}_wheel_trans">
+      <type>transmission_interface/SimpleTransmission</type>
+      <actuator name="joint_${suffix}_wheel_motor">
+        <mechanicalReduction>1</mechanicalReduction>
+      </actuator>
+      <joint name="joint_${suffix}">
+        <hardwareInterface>hardware_interface/VelocityJointInterface</hardwareInterface>
+      </joint>
+    </transmission>
+    <!--Some extra Gazebo details-->
+    <gazebo reference="link_${suffix}">
+      <mu1 value="200.0"/>
+      <mu2 value="100.0"/>
+      <kp value="10000000.0" />
+      <kd value="1.0" />
+      <material>Gazebo/Blue</material>
+    </gazebo>
   </xacro:macro>
   <!--Links-->
@@ -65,4 +83,7 @@
       <inertia ixx="4.05" ixy="0" ixz="0" iyy="9.82" iyz="0" izz="12.25"/>
     </inertial>
+    <gazebo>
+      <material>Gazebo/Grey</material>
+    </gazebo>
   </link>
   <!--wheel/joint_0-->
@@ -74,5 +95,5 @@
   <!--wheel/joint_3-->
   <xacro:wheel suffix="3" reflect_x="-1" reflect_y="-1" reflect_z="-1" />
-	<!--Plugin ties Gazebo to ROS-->
+	<!--Gazebo plugin for ROS controls-->
 	<gazebo>
 		<plugin name="gazebo_ros_control" filename="libgazebo_ros_control.so">

Commit message: Add files via upload

File: backups/lunarbot/urdf/lunarbot.urdf.xacro (robot description, xacro)
@@ -211,4 +211,27 @@
     <material>Gazebo/Blue</material>
   </gazebo>
+  <!--<link name="auger">
+    <visual>
+      <origin rpy="0 0 0" xyz="0 0 0"/>
+      <geometry>
+         <mesh filename="package://lunarbot/meshes/auger.dae"/>
+      </geometry>
+    </visual>
+  </link>
+  <collision>
+    <geometry>
+      <cylinder length="1.3" radius=".2"/>
+    </geometry>
+  </collision>
+  <inertial>
+    <mass value="33"/>
+    <inertia ixx="4.73" ixy="0" ixz="0" iyy="4.73" iyz="0" izz=".165"/>
+  </inertial>
+  <joint name="auger" type="continuous">
+    <parent link="base_link"/>
+    <child link="auger"/>
+    <axis xyz="0 0 1"/>
+    <origin rpy="0 0 0" xyz="0 0 1"/>
+  </joint>-->
   <!--Gazebo plugin for ROS controls-->
   <gazebo>

File: backups/lunarbot/urdf/lunarbot2.urdf (robot description, URDF)
Before this commit: robot Roberto_MkI, 5 links, 4 joints
Links:
- added link auger, mass 33; collision cylinder length=1.05 radius=.18; visual mesh filename=package://lunarbot/meshes/auger.stl
- added link link_4; visual box size=.05 .1 .8
- added link link_5; visual box size=.1 .1 .3
- link base_link: geometry collision box size=1.5 0.8 .3; visual mesh filename=package://lunarbot/meshes/base_link2.stl
- link link_0: geometry collision cylinder length=0.15 radius=0.3; visual cylinder length=0.15 radius=0.3
- link link_1: geometry collision cylinder length=0.15 radius=0.3; visual cylinder length=0.15 radius=0.3
- link link_2: geometry collision cylinder length=0.15 radius=0.3; visual cylinder length=0.15 radius=0.3
- link link_3: geometry collision cylinder length=0.15 radius=0.3; visual cylinder length=0.15 radius=0.3
Joints:
- added joint auger_joint: type continuous, parent link_5, child auger, origin xyz=.23 0 0, axis 0 0 1
- added joint joint_4: type fixed, parent base_link, child link_4, origin xyz=-.25 0 -.05 rpy=0 -.85 0
- added joint joint_5: type prismatic, parent link_4, child link_5, origin xyz=0 0 .65, axis 0 0 1, limit lower=-.55 upper=0 effort=1000 velocity=.5
- joint joint_0: origin xyz=0.3 0.375 -0.075 rpy=0 0 0 -> xyz=0.6 0.475 -0.075
- joint joint_1: origin xyz=0.3 -0.375 -0.075 rpy=0 0 0 -> xyz=0.6 -0.475 -0.075
- joint joint_2: origin xyz=-0.3 0.375 -0.075 rpy=0 0 0 -> xyz=-0.6 0.475 -0.075
- joint joint_3: origin xyz=-0.3 -0.375 -0.075 rpy=0 0 0 -> xyz=-0.6 -0.475 -0.075

File: backups/lunarbot/urdf/lunarbot2.xacro (robot description, xacro)
@@ -1,5 +1,5 @@
 <?xml version="1.0"?>
 <!--Name of robot-->
-<robot xmlns:xacro="http://www.ros.org/wiki/xacro" name="Roberto_MkI">
+<robot xmlns:xacro="http://www.ros.org/wiki/xacro" name="Roberto_MkII">
   <!--Naming Materials-->
   <material name="blue">
@@ -9,10 +9,16 @@
     <color rgba="1 1 1 1"/>
   </material>
+  <material name="black">
+    <color rgba="0 0 0 1"/>
+  </material>
+  <material name="green">
+    <color rgba="0 1 0 1"/>
+  </material>
   <!--Xacro Macros-->
   <!--Body Macros-->
-  <xacro:property name="body_size" value="1.0 0.6 0.3" />
+  <xacro:property name="body_size" value="1.5 0.8 .3" />
   <!--Wheel Macros-->
   <xacro:property name="wheel_len" value=".15" />
-  <xacro:property name="wheel_rad" value=".2" />
+  <xacro:property name="wheel_rad" value=".3" />
   <xacro:property name="wheel_origin" value="1.57075 0 0" />
   <xacro:macro name="wheel" params="suffix reflect_x reflect_y reflect_z">
@@ -40,5 +46,5 @@
       <child link="link_${suffix}"/>
       <axis xyz="0 1 0"/>
-      <origin rpy="0 0 0" xyz="${reflect_x * 0.3} ${reflect_y * 0.375} ${reflect_z * 0.075}"/>
+      <origin xyz="${reflect_x * 0.6} ${reflect_y * 0.475} ${reflect_z * 0.075}"/>
     </joint>
     <!--Connects Gazebo to ROS Controls-->
@@ -49,5 +55,6 @@
       </actuator>
       <joint name="joint_${suffix}">
-        <hardwareInterface>hardware_interface/VelocityJointInterface</hardwareInterface>
+        <hardwareInterface>hardware_interface/VelocityJointInterface
+        </hardwareInterface>
       </joint>
     </transmission>
@@ -56,6 +63,6 @@
       <mu1 value="200.0"/>
       <mu2 value="100.0"/>
-      <kp value="10000000.0" />
-      <kd value="1.0" />
+      <kp value="10000000.0"/>
+      <kd value="1.0"/>
       <material>Gazebo/Blue</material>
     </gazebo>
@@ -67,7 +74,7 @@
     <visual>
       <geometry>
-        <box size="${body_size}"/>
+        <mesh filename="package://lunarbot/meshes/base_link2.stl"/>
       </geometry>
-        <material name="white"/>
+      <material name="white"/>
     </visual>
     <!--Collision-->
@@ -95,32 +102,85 @@
   <!--wheel/joint_3-->
   <xacro:wheel suffix="3" reflect_x="-1" reflect_y="-1" reflect_z="-1" />
-  <!--<link name="auger">
+  <link name="auger">
     <visual>
-      <origin rpy="0 0 0" xyz="0 0 0"/>
+      <origin xyz="0 0 -1.2"/>
       <geometry>
-         <mesh filename="package://lunarbot/meshes/auger.dae"/>
+         <mesh filename="package://lunarbot/meshes/auger.stl"/>
       </geometry>
+      <material name="black"/>
+    </visual>
+    <collision>
+      <geometry>
+        <cylinder length="1.05" radius=".18"/>
+      </geometry>
+      <origin xyz="0 0 -.565"/>
+    </collision>
+    <inertial>
+      <mass value="33"/>
+      <inertia ixx="4.73" ixy="0" ixz="0" iyy="4.73" iyz="0" izz=".165"/>
+    </inertial>
+  </link>
+  <joint name="auger_joint" type="continuous">
+    <parent link="link_5"/>
+    <child link="auger"/>
+    <axis xyz="0 0 1"/>
+    <origin xyz=".23 0 0"/>
+  </joint>
+  <transmission name="auger_joint_trans">
+    <type>transmission_interface/SimpleTransmission</type>
+    <actuator name="auger_joint_motor">
+      <mechanicalReduction>1</mechanicalReduction>
+    </actuator>
+    <joint name="auger_joint">
+      <hardwareInterface>hardware_interface/VelocityJointInterface
+      </hardwareInterface>
+    </joint>
+  </transmission>
+  <link name="link_4">
+    <visual>
+      <geometry>
+        <box size=".05 .1 .8"/>
+      </geometry>
+      <origin xyz="0 0 .3"/>
+      <material name="green"/>
+    </visual>
+    <gazebo>
+      <material>Gazebo/Yellow</material>
+    </gazebo>
+  </link>
+  <joint name="joint_4" type="fixed">
+    <parent link="base_link"/>
+    <child link="link_4"/>
+    <origin rpy="0 -.85 0" xyz="-.25 0 -.05"/>
+  </joint>
+  <link name="link_5">
+    <visual>
+      <geometry>
+        <box size=".1 .1 .3"/>
+      </geometry>
+      <origin rpy="0 1.575 0" xyz=".15 0 0"/>
+      <material name="blue"/>
     </visual>
   </link>
-  <collision>
-    <geometry>
-      <cylinder length="1.3" radius=".2"/>
-    </geometry>
-  </collision>
-  <inertial>
-    <mass value="33"/>
-    <inertia ixx="4.73" ixy="0" ixz="0" iyy="4.73" iyz="0" izz=".165"/>
-  </inertial>
-  <joint name="auger" type="continuous">
-    <parent link="base_link"/>
-    <child link="auger"/>
+  <joint name="joint_5" type="prismatic">
+    <parent link="link_4"/>
+    <child link="link_5"/>
     <axis xyz="0 0 1"/>
-    <origin rpy="0 0 0" xyz="0 0 1"/>
-  </joint>-->
+    <limit effort="1000" lower="-.55" upper="0" velocity=".5"/>
+    <origin xyz="0 0 .65"/>
+  </joint>
+  <transmission name="joint_5_trans">
+    <type>transmission_interface/SimpleTransmission</type>
+    <actuator name="joint_5_motor">
+      <mechanicalReduction>1</mechanicalReduction>
+    </actuator>
+    <joint name="joint_5">
+      <hardwareInterface>hardware_interface/EffortJointInterface
+      </hardwareInterface>
+    </joint>
+  </transmission>
 	<!--Gazebo plugin for ROS controls-->
 	<gazebo>
-		<plugin name="gazebo_ros_control" filename="libgazebo_ros_control.so">
-			<robotNamespace>/</robotNamespace>
-		</plugin>
+	  <plugin name="gazebo_ros_control" filename="libgazebo_ros_control.so"/>
 	</gazebo>
 </robot>
